File: Goyala Fang PCB/Goyala Fang PCB.kicad_sch (KiCad schematic)
At the start: 9 parts, among them J1 Input Battery, J2 Conn_01x06, U3 L298N, U5 MPU-6050, U6 INA219AxD

Commit message: [Feat] Added App
Parts:
- J1: footprint (none) -> Connector_PinSocket_2.54mm:PinSocket_1x02_P2.54mm_Vertical
- U3: footprint Connector_PinSocket_2.54mm:PinSocket_1x04_P2.54mm_Vertical -> Connector_PinSocket_2.54mm:PinSocket_1x06_P2.54mm_Vertical
- U4: footprint Connector_PinSocket_2.54mm:PinSocket_1x03_P2.54mm_Vertical -> Connector_PinSocket_2.54mm:PinSocket_1x04_P2.54mm_Vertical
Connections:
- net GND: now also U1.6 (GND), U4.4 (GND); no longer U1.3 (GND), U4.2 (GND)
- net ena: now also A1.13 (D10); no longer A1.11 (D8)
- net in1: now also A1.6 (D3); no longer A1.13 (D10), A1.7 (D4)
- net in2: now also A1.5 (D2); no longer A1.12 (D9)
- net at A1.1 (D1/TX): now also U4.2 (Rx); no longer U4.4 (Rx)
- net at A1.15 (D12): now also J2.5 (Pin_3); no longer J2.3 (Pin_3)
- net at A1.19 (A0): now also J2.3 (Pin_5); no longer J2.5 (Pin_5)
- net rx2: now reaches U1.5 (TXD)
- net rx2: now also A1.12 (D9); no longer A1.5 (D2)
- net tx2: now reaches U1.4 (RXD)
- net tx2: now also A1.11 (D8); no longer A1.6 (D3)
